Commit message: feat(urdf_tools): rich warehouse 3D structure + fix scan cloud rendering
warehouse_world.urdf — complete rewrite with 44 primitive geometry blocks:
  • Floor slab (50×30×0.1 m) and roof slab (50×30×0.25 m)
  • 4 outer walls (6 m tall, 0.3 m thick)
  • 3×3 grid of structural columns (cylinder r=0.18, h=6)
  • 6 overhead beams: 3 spanning Y at x=10,25,40 and
    3 spanning X at y=7,15,23 (at z≈5.65–5.70 m)
  • 20 storage-rack bays in 4 rows (amber wireframe) placed in the
    aisles between column lines
  • 3 loading-dock portal frames (yellow) on the south wall
  Removed: mesh-only "structure" link and near-transparent scene_bounds
  box (both were invisible in wireframe rendering).

05_sub_viewer.py:
  _draw_urdf_3d_static — tint wireframe edge colour from each element's
    URDF material rgba so walls, columns, racks and beams are visually
    distinct instead of uniform _WORLD_EC.

  live3d — fix scan point cloud not rendering:
    • Initialise scan_scat with one off-screen seed point (c=[0.0])
      instead of empty c=[] so the internal colormap state is set up.
    • Replace set_array()/set_clim() with explicit plt.cm.plasma()
      colour computation to bypass the empty-init state issue.
    • Fix axis limits: use per-axis tight bounds (xlim, ylim follow URDF
      extents; zlim = -0.5…zmax+0.5) instead of symmetric expansion
      that inflated z-range to ~30 m, pushing scan hits at z=0.05 to
      the invisible bottom strip.
    • Set view_init(elev=32, azim=-52) for a clear angled overview.

Co-Authored-By: Claude Sonnet 4.6 <noreply@anthropic.com>
Claude-Session: https://claude.ai/code/session_01EgxXHGj54sJxpHeH1itWRo

File: urdf_tools/examples/models/warehouse_world.urdf (robot description, URDF)
Before this commit: robot warehouse_world, 8 links, 7 joints
Links:
- removed link pillar_nw
- removed link pillar_sw
- removed link scene_bounds
- removed link structure
- added link beam_x_y15; visual box size=50 0.30 0.35
- added link beam_x_y23; visual box size=50 0.30 0.35
- added link beam_x_y7; visual box size=50 0.30 0.35
- added link beam_y_x10; visual box size=0.30 30 0.40
- added link beam_y_x25; visual box size=0.30 30 0.40
- added link beam_y_x40; visual box size=0.30 30 0.40
- added link col_r1c1; visual cylinder length=6 radius=0.18
- added link col_r1c2; visual cylinder length=6 radius=0.18
- added link col_r1c3; visual cylinder length=6 radius=0.18
- added link col_r2c1; visual cylinder length=6 radius=0.18
- added link col_r2c2; visual cylinder length=6 radius=0.18
- added link col_r2c3; visual cylinder length=6 radius=0.18
- added link col_r3c1; visual cylinder length=6 radius=0.18
- added link col_r3c2; visual cylinder length=6 radius=0.18
- added link col_r3c3; visual cylinder length=6 radius=0.18
- added link floor; visual box size=50 30 0.1
- added link rack_r1b1; visual box size=8 1.2 4.2
- added link rack_r1b2; visual box size=8 1.2 4.2
- added link rack_r1b3; visual box size=8 1.2 4.2
- added link rack_r1b4; visual box size=8 1.2 4.2
- added link rack_r1b5; visual box size=8 1.2 4.2
- added link rack_r2b1; visual box size=8 1.2 4.2
- added link rack_r2b2; visual box size=8 1.2 4.2
- added link rack_r2b3; visual box size=8 1.2 4.2
- added link rack_r2b4; visual box size=8 1.2 4.2
- added link rack_r2b5; visual box size=8 1.2 4.2
- added link rack_r3b1; visual box size=8 1.2 4.2
- added link rack_r3b2; visual box size=8 1.2 4.2
- added link rack_r3b3; visual box size=8 1.2 4.2
- added link rack_r3b4; visual box size=8 1.2 4.2
- added link rack_r3b5; visual box size=8 1.2 4.2
- added link rack_r4b1; visual box size=8 1.2 4.2
- added link rack_r4b2; visual box size=8 1.2 4.2
- added link rack_r4b3; visual box size=8 1.2 4.2
- added link rack_r4b4; visual box size=8 1.2 4.2
- added link rack_r4b5; visual box size=8 1.2 4.2
- added link roof; visual box size=50 30 0.25
- added link wall_east; visual box size=0.3 30 6
- added link wall_north; visual box size=50 0.3 6
- added link wall_south; visual box size=50 0.3 6
- added link wall_west; visual box size=0.3 30 6
Joints:
- removed joint world_to_bounds
- removed joint world_to_pillar_nw
- removed joint world_to_pillar_sw
- removed joint world_to_structure
- added joint j_beam_x_y15: type fixed, parent world, child beam_x_y15, origin xyz=0 15 0 rpy=0 0 0
- added joint j_beam_x_y23: type fixed, parent world, child beam_x_y23, origin xyz=0 23 0 rpy=0 0 0
- added joint j_beam_x_y7: type fixed, parent world, child beam_x_y7, origin xyz=0 7 0 rpy=0 0 0
- added joint j_beam_y_x10: type fixed, parent world, child beam_y_x10, origin xyz=10 0 0 rpy=0 0 0
- added joint j_beam_y_x25: type fixed, parent world, child beam_y_x25, origin xyz=25 0 0 rpy=0 0 0
- added joint j_beam_y_x40: type fixed, parent world, child beam_y_x40, origin xyz=40 0 0 rpy=0 0 0
- added joint j_col_r1c1: type fixed, parent world, child col_r1c1, origin xyz=10 7 0 rpy=0 0 0
- added joint j_col_r1c2: type fixed, parent world, child col_r1c2, origin xyz=25 7 0 rpy=0 0 0
- added joint j_col_r1c3: type fixed, parent world, child col_r1c3, origin xyz=40 7 0 rpy=0 0 0
- added joint j_col_r2c1: type fixed, parent world, child col_r2c1, origin xyz=10 15 0 rpy=0 0 0
- added joint j_col_r2c2: type fixed, parent world, child col_r2c2, origin xyz=25 15 0 rpy=0 0 0
- added joint j_col_r2c3: type fixed, parent world, child col_r2c3, origin xyz=40 15 0 rpy=0 0 0
- added joint j_col_r3c1: type fixed, parent world, child col_r3c1, origin xyz=10 23 0 rpy=0 0 0
- added joint j_col_r3c2: type fixed, parent world, child col_r3c2, origin xyz=25 23 0 rpy=0 0 0
- added joint j_col_r3c3: type fixed, parent world, child col_r3c3, origin xyz=40 23 0 rpy=0 0 0
- added joint j_floor: type fixed, parent world, child floor, origin xyz=0 0 0 rpy=0 0 0
- added joint j_rack_r1b1: type fixed, parent world, child rack_r1b1, origin xyz=7 3.0 0 rpy=0 0 0
- added joint j_rack_r1b2: type fixed, parent world, child rack_r1b2, origin xyz=16 3.0 0 rpy=0 0 0
- added joint j_rack_r1b3: type fixed, parent world, child rack_r1b3, origin xyz=25 3.0 0 rpy=0 0 0
- added joint j_rack_r1b4: type fixed, parent world, child rack_r1b4, origin xyz=34 3.0 0 rpy=0 0 0
- added joint j_rack_r1b5: type fixed, parent world, child rack_r1b5, origin xyz=43 3.0 0 rpy=0 0 0
- added joint j_rack_r2b1: type fixed, parent world, child rack_r2b1, origin xyz=7 11.0 0 rpy=0 0 0
- added joint j_rack_r2b2: type fixed, parent world, child rack_r2b2, origin xyz=16 11.0 0 rpy=0 0 0
- added joint j_rack_r2b3: type fixed, parent world, child rack_r2b3, origin xyz=25 11.0 0 rpy=0 0 0
- added joint j_rack_r2b4: type fixed, parent world, child rack_r2b4, origin xyz=34 11.0 0 rpy=0 0 0
- added joint j_rack_r2b5: type fixed, parent world, child rack_r2b5, origin xyz=43 11.0 0 rpy=0 0 0
- added joint j_rack_r3b1: type fixed, parent world, child rack_r3b1, origin xyz=7 19.0 0 rpy=0 0 0
- added joint j_rack_r3b2: type fixed, parent world, child rack_r3b2, origin xyz=16 19.0 0 rpy=0 0 0
- added joint j_rack_r3b3: type fixed, parent world, child rack_r3b3, origin xyz=25 19.0 0 rpy=0 0 0
- added joint j_rack_r3b4: type fixed, parent world, child rack_r3b4, origin xyz=34 19.0 0 rpy=0 0 0
- added joint j_rack_r3b5: type fixed, parent world, child rack_r3b5, origin xyz=43 19.0 0 rpy=0 0 0
- added joint j_rack_r4b1: type fixed, parent world, child rack_r4b1, origin xyz=7 27.0 0 rpy=0 0 0
- added joint j_rack_r4b2: type fixed, parent world, child rack_r4b2, origin xyz=16 27.0 0 rpy=0 0 0
- added joint j_rack_r4b3: type fixed, parent world, child rack_r4b3, origin xyz=25 27.0 0 rpy=0 0 0
- added joint j_rack_r4b4: type fixed, parent world, child rack_r4b4, origin xyz=34 27.0 0 rpy=0 0 0
- added joint j_rack_r4b5: type fixed, parent world, child rack_r4b5, origin xyz=43 27.0 0 rpy=0 0 0
- added joint j_roof: type fixed, parent world, child roof, origin xyz=0 0 0 rpy=0 0 0
- added joint j_wall_east: type fixed, parent world, child wall_east, origin xyz=0 0 0 rpy=0 0 0
- added joint j_wall_north: type fixed, parent world, child wall_north, origin xyz=0 0 0 rpy=0 0 0
- added joint j_wall_south: type fixed, parent world, child wall_south, origin xyz=0 0 0 rpy=0 0 0
- added joint j_wall_west: type fixed, parent world, child wall_west, origin xyz=0 0 0 rpy=0 0 0
